File: me.kicad_sch (KiCad schematic)
At the start: 15 parts, among them M1 Motor_DC, Q1 AO3400A, SW1 SW_Push, SW2 SW_Push, SW3 SW_Push, SW4 SW_Push, SW5 SW_Push, SW6 SW_Push, U1 XIAO-RP2040-DIP

Commit message: erwovnojerwnhvonwejvew
wrjgvwjngvloekr3w
Parts:
- removed D1: SK6812MINI, LED_SMD:LED_SK6812MINI_PLCC4_3.5x3.5mm_P1.75mm, symbol LED:SK6812MINI
- C1: footprint (none) -> Capacitor_SMD:C_0603_1608Metric
- M1: footprint (none) -> Connector_PinHeader_2.54mm:PinHeader_1x02_P2.54mm_Vertical
- R1: footprint (none) -> Resistor_SMD:R_0603_1608Metric
Connections:
- net +5V: now also C1.2, D4.2 (A)
- net at U1.1 (GPIO26/ADC0/A0): now also R1.1
- net at U1.11 (GPIO3/MOSI): now also D3.3 (DIN); no longer SW4.2
- net at U1.3 (GPIO28/ADC2/A2): now also SW4.2
- net at D4.1 (K): now also C1.1, M1.2 (-), Q1.3 (D)
- net at R1.2: now also Q1.1 (G)
Other:
- moved on the sheet: C1, D4, M1, Q1, R1, SW4, SW5

Commit message: aiehf
Connections:
- no-connect marks 0 -> 5
Other:
- moved on the sheet: M1
Changed lines of the file:
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@@
+	)
+	(junction
+		(at 55.88 87.63)
+		(diameter 0)
+		(color 0 0 0 0)
 	)
 	(junction
@@
 	)
 	(junction
-		(at 55.88 87.63)
-		(diameter 0)
-		(color 0 0 0 0)
-	)
-	(junction
-		(at 119.38 41.91)
-		(diameter 0)
-		(color 0 0 0 0)
-	)
-	(junction
 		(at 55.88 116.84)
 		(diameter 0)
@@
 	)
 	(junction
-		(at 158.75 48.26)
+		(at 158.75 46.99)
 		(diameter 0)
 		(color 0 0 0 0)
@@
 		(color 0 0 0 0)
 	)
+	(junction
+		(at 119.38 40.64)
+		(diameter 0)
+		(color 0 0 0 0)
+	)
+	(no_connect
+		(at 96.52 74.93)
+	)
+	(no_connect
+		(at 96.52 86.36)
+	)
+	(no_connect
+		(at 96.52 82.55)
+	)
+	(no_connect
+		(at 132.08 78.74)
+	)
+	(no_connect
+		(at 127 49.53)
+	)
 	(wire
 		(pts
@@
 	(wire
 		(pts
+			(xy 149.86 46.99) (xy 158.75 46.99)
+		)
+		(stroke
+			(width 0)
+			(type default)
+		)
+	)
+	(wire
+		(pts
 			(xy 66.04 154.94) (xy 38.1 154.94)
 		)
@@
 	(wire
 		(pts
-			(xy 158.75 41.91) (xy 158.75 48.26)
-		)
-		(stroke
-			(width 0)
-			(type default)
-		)
-	)
-	(wire
-		(pts
 			(xy 55.88 105.41) (xy 55.88 116.84)
 		)
@@
 	(wire
 		(pts
-			(xy 149.86 50.8) (xy 149.86 48.26)
+			(xy 99.06 58.42) (xy 119.38 58.42)
+		)
+		(stroke
+			(width 0)
+			(type default)
+		)
+	)
+	(wire
+		(pts
+			(xy 149.86 46.99) (xy 149.86 50.8)
+		)
+		(stroke
+			(width 0)
+			(type default)
+		)
+	)
+	(wire
+		(pts
+			(xy 99.06 41.91) (xy 115.57 41.91)
+		)
+		(stroke
+			(width 0)
+			(type default)
+		)
+	)
+	(wire
+		(pts
+			(xy 158.75 62.23) (xy 158.75 60.96)
+		)
+		(stroke
+			(width 0)
+			(type default)
+		)
+	)
+	(wire
+		(pts
+			(xy 115.57 41.91) (xy 115.57 40.64)
 		)
 		(stroke
@@
 	(wire
 		(pts
-			(xy 99.06 58.42) (xy 119.38 58.42)
-		)
-		(stroke
-			(width 0)
-			(type default)
-		)
-	)
-	(wire
-		(pts
 			(xy 80.01 116.84) (xy 68.58 116.84)
 		)
@@
 	(wire
 		(pts
-			(xy 119.38 58.42) (xy 119.38 57.15)
-		)
-		(stroke
-			(width 0)
-			(type default)
-		)
-	)
-	(wire
-		(pts
-			(xy 158.75 60.96) (xy 158.75 62.23)
-		)
-		(stroke
-			(width 0)
-			(type default)
-		)
-	)
-	(wire
-		(pts
 			(xy 76.2 90.17) (xy 96.52 90.17)
 		)
@@
 	(wire
 		(pts
-			(xy 149.86 48.26) (xy 158.75 48.26)
-		)
-		(stroke
-			(width 0)
-			(type default)
-		)
-	)
-	(wire
-		(pts
 			(xy 130.81 93.98) (xy 130.81 101.6)
 		)
@@
 	(wire
 		(pts
+			(xy 115.57 40.64) (xy 119.38 40.64)
+		)
+		(stroke
+			(width 0)
+			(type default)
+		)
+	)
+	(wire
+		(pts
 			(xy 83.82 59.69) (xy 85.09 59.69)
 		)
@@
 	(wire
 		(pts
+			(xy 119.38 58.42) (xy 119.38 59.69)
+		)
+		(stroke
+			(width 0)
+			(type default)
+		)
+	)
+	(wire
+		(pts
 			(xy 149.86 66.04) (xy 149.86 67.31)
 		)
@@
 	(wire
 		(pts
-			(xy 99.06 41.91) (xy 119.38 41.91)
+			(xy 173.99 46.99) (xy 173.99 48.26)
+		)
+		(stroke
+			(width 0)
+			(type default)
+		)
+	)
+	(wire
+		(pts
+			(xy 119.38 40.64) (xy 119.38 41.91)
 		)
 		(stroke
@@
 	(wire
 		(pts
-			(xy 158.75 48.26) (xy 173.99 48.26)
-		)
-		(stroke
-			(width 0)
-			(type default)
-		)
-	)
-	(wire
-		(pts
 			(xy 85.09 78.74) (xy 96.52 78.74)
 		)
@@
 	(wire
 		(pts
+			(xy 119.38 35.56) (xy 119.38 40.64)
+		)
+		(stroke
+			(width 0)
+			(type default)
+		)
+	)
+	(wire
+		(pts
 			(xy 96.52 66.04) (xy 96.52 71.12)
 		)
@@
 	(wire
 		(pts
-			(xy 158.75 49.53) (xy 158.75 48.26)
-		)
-		(stroke
-			(width 0)
-			(type default)
-		)
-	)
-	(wire
-		(pts
 			(xy 38.1 154.94) (xy 38.1 63.5)
 		)
@@
 	(wire
 		(pts
+			(xy 158.75 41.91) (xy 158.75 46.99)
+		)
+		(stroke
+			(width 0)
+			(type default)
+		)
+	)
+	(wire
+		(pts
 			(xy 66.04 87.63) (xy 66.04 104.14)
 		)
@@
 	(wire
 		(pts
+			(xy 158.75 46.99) (xy 173.99 46.99)
+		)
+		(stroke
+			(width 0)
+			(type default)
+		)
+	)
+	(wire
+		(pts
 			(xy 46.99 69.85) (xy 71.12 69.85)
 		)
@@
 	(wire
 		(pts
+			(xy 158.75 59.69) (xy 158.75 60.96)
+		)
+		(stroke
+			(width 0)
+			(type default)
+		)
+	)
+	(wire
+		(pts
 			(xy 46.99 139.7) (xy 46.99 69.85)
+		)
+		(stroke
+			(width 0)
+			(type default)
+		)
+	)
+	(wire
+		(pts
+			(xy 119.38 57.15) (xy 119.38 58.42)
 		)
 		(stroke
@@
 	(symbol
 		(lib_id "power:+5V")
-		(at 119.38 41.91 0)
+		(at 119.38 35.56 0)
 		(unit 1)
 		(exclude_from_sim no)
@@
 		(fields_autoplaced yes)
 		(property "Reference" "#PWR02"
-			(at 119.38 45.72 0)
+			(at 119.38 39.37 0)
 			(effects
 				(font
@@
 		)
 		(property "Value" "+5V"
-			(at 119.38 36.83 0)
+			(at 119.38 30.48 0)
 			(effects
 				(font
@@
 		)
 		(property "Footprint" ""
-			(at 119.38 41.91 0)
+			(at 119.38 35.56 0)
 			(effects
 				(font
@@
 		)
 		(property "Datasheet" ""
-			(at 119.38 41.91 0)
+			(at 119.38 35.56 0)
 			(effects
 				(font
@@
 		)
 		(property "Description" "Power symbol creates a global label with name \"+5V\""
-			(at 119.38 41.91 0)
+			(at 119.38 35.56 0)
 			(effects
 				(font
@@
 	(symbol
 		(lib_id "Motor:Motor_DC")
-		(at 158.75 53.34 0)
+		(at 158.75 52.07 0)
 		(unit 1)
 		(exclude_from_sim no)
@@
 		(fields_autoplaced yes)
 		(property "Reference" "M1"
-			(at 163.83 54.6099 0)
+			(at 163.83 53.3399 0)
 			(effects
 				(font
@@
 		)
 		(property "Value" "Motor_DC"
-			(at 163.83 57.1499 0)
+			(at 163.83 55.8799 0)
 			(effects
 				(font
@@
 		)
 		(property "Footprint" "Connector_PinHeader_2.54mm:PinHeader_1x02_P2.54mm_Vertical"
-			(at 158.75 55.626 0)
+			(at 158.75 54.356 0)
 			(effects
 				(font
@@
 		)
 		(property "Datasheet" "~"
-			(at 158.75 55.626 0)
+			(at 158.75 54.356 0)
 			(effects
 				(font
@@
 		)
 		(property "Description" "DC Motor"
-			(at 158.75 53.34 0)
+			(at 158.75 52.07 0)
 			(effects
 				(font
@@
 	(symbol
 		(lib_id "power:GND")
-		(at 119.38 58.42 0)
+		(at 119.38 59.69 0)
 		(unit 1)
 		(exclude_from_sim no)
@@
 		(dnp no)
 		(property "Reference" "#PWR01"
-			(at 119.38 64.77 0)
+			(at 119.38 66.04 0)
 			(effects
 				(font
@@
 		)
 		(property "Value" "GND"
-			(at 119.126 62.23 0)
+			(at 119.126 63.5 0)
 			(effects
 				(font
@@
 		)
 		(property "Footprint" ""
-			(at 119.38 58.42 0)
+			(at 119.38 59.69 0)
 			(effects
 				(font
@@
 		)
 		(property "Datasheet" ""
-			(at 119.38 58.42 0)
+			(at 119.38 59.69 0)
 			(effects
 				(font
@@
 		)
 		(property "Description" "Power symbol creates a global label with name \"GND\" , ground"
-			(at 119.38 58.42 0)
-			(effects
-				(font
+			(at 119.38 59.69 0)
+			(effects
+				(font

Commit message: houweg
Changed lines of the file:
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@@
+	)
+	(junction
+		(at 119.38 38.1)
+		(diameter 0)
+		(color 0 0 0 0)
 	)
 	(junction
@@
 	(wire
 		(pts
+			(xy 121.92 38.1) (xy 119.38 38.1)
+		)
+		(stroke
+			(width 0)
+			(type default)
+		)
+	)
+	(wire
+		(pts
 			(xy 80.01 139.7) (xy 46.99 139.7)
 		)
@@
 	(wire
 		(pts
-			(xy 119.38 35.56) (xy 119.38 40.64)
+			(xy 119.38 35.56) (xy 119.38 38.1)
 		)
 		(stroke
@@
 		(pts
 			(xy 137.16 90.17) (xy 132.08 90.17)
+		)
+		(stroke
+			(width 0)
+			(type default)
+		)
+	)
+	(wire
+		(pts
+			(xy 119.38 38.1) (xy 119.38 40.64)
 		)
 		(stroke
@@
 	)
 	(symbol
+		(lib_id "power:PWR_FLAG")
+		(at 119.38 58.42 270)
+		(unit 1)
+		(exclude_from_sim no)
+		(in_bom yes)
+		(on_board yes)
+		(dnp no)
+		(fields_autoplaced yes)
+		(property "Reference" "#FLG02"
+			(at 121.285 58.42 0)
+			(effects
+				(font
+					(size 1.27 1.27)
+				)
+				(hide yes)
+			)
+		)
+		(property "Value" "PWR_FLAG"
+			(at 123.19 58.4199 90)
+			(effects
+				(font
+					(size 1.27 1.27)
+				)
+				(justify left)
+			)
+		)
+		(property "Footprint" ""
+			(at 119.38 58.42 0)
+			(effects
+				(font
+					(size 1.27 1.27)
+				)
+				(hide yes)
+			)
+		)
+		(property "Datasheet" "~"
+			(at 119.38 58.42 0)
+			(effects
+				(font
+					(size 1.27 1.27)
+				)
+				(hide yes)
+			)
+		)
+		(property "Description" "Special symbol for telling ERC where power comes from"
+			(at 119.38 58.42 0)
+			(effects
+				(font
+					(size 1.27 1.27)
+				)
+				(hide yes)
+			)
+		)
+		(pin "1"
+		)
+		(instances
+			(project ""
+				(path "/b846a21e-b21a-4d67-8cb5-5d89945714aa"
+					(reference "#FLG02")
+					(unit 1)
+				)
+			)
+		)
+	)
+	(symbol
 		(lib_id "Device:R")
 		(at 173.99 52.07 180)
@@
 					(unit 1)
 				)
+			)
+		)
+	)
+	(symbol
+		(lib_id "power:PWR_FLAG")
+		(at 121.92 38.1 270)
+		(unit 1)
+		(exclude_from_sim no)
+		(in_bom yes)
+		(on_board yes)
+		(dnp no)
+		(fields_autoplaced yes)
+		(property "Reference" "#FLG01"
+			(at 123.825 38.1 0)
+			(effects
+				(font
+					(size 1.27 1.27)
+				)
+				(hide yes)
+			)
+		)
+		(property "Value" "PWR_FLAG"
+			(at 125.73 38.0999 90)
+			(effects
+				(font
+					(size 1.27 1.27)
+				)
+				(justify left)
+			)
+		)
+		(property "Footprint" ""
+			(at 121.92 38.1 0)
+			(effects
+				(font
+					(size 1.27 1.27)
+				)
+				(hide yes)
+			)
+		)
+		(property "Datasheet" "~"
+			(at 121.92 38.1 0)
+			(effects
+				(font
+					(size 1.27 1.27)
+				)
+				(hide yes)
+			)
+		)
+		(property "Description" "Special symbol for telling ERC where power comes from"
+			(at 121.92 38.1 0)
+			(effects
+				(font
+					(size 1.27 1.27)
+				)
+				(hide yes)
+			)
+		)
+		(pin "1"
+		)
+		(instances
+			(project ""
+				(path "/b846a21e-b21a-4d67-8cb5-5d89945714aa"
+					(reference "#FLG01")
+					(unit 1)
+				)
