File: PCB/me.kicad_pcb (KiCad board)
At the start: 2 copper layers, 166.7 x 154.5 mm, 14 parts, among them M1 Motor_DC, Q1 AO3400A, SW1 SW_Push, SW2 SW_Push, SW3 SW_Push, SW4 SW_Push, SW5 SW_Push, SW6 SW_Push, U1 XIAO-RP2040-DIP

Commit message: please
Parts:
- moved R1 49.7 mm to (173.8, 126.2)
- moved D4 45.4 mm to (181.0, 126.2)
- moved D2 43.9 mm to (138.1, 133.3)
- moved Q1 43.3 mm to (177.2, 132.4)
- moved D3 40.2 mm to (138.1, 128.6)
- moved C1 37.7 mm to (200.0, 109.5)
- moved M1 37.3 mm to (188.1, 111.8)
- moved U1 34.0 mm to (156.6, 134.9)
- moved SW1 13.5 mm to (126.4, 73.5)
- moved SW2 12.1 mm to (118.9, 99.7)
- moved SW4 10.3 mm to (157.0, 94.9)
- moved SW6 9.90 mm to (138.0, 97.3)
- moved SW3 8.59 mm to (145.4, 71.1)
- moved SW5 4.77 mm to (164.8, 68.7)
Routing:
- net GND: track 443.3 -> 252.7 mm, vias 0 -> 1
- net Net-(U1-GPIO28/ADC2/A2): track 143.0 -> 47.6 mm
- net Net-(U1-GPIO7/SCL): track 143.7 -> 72.9 mm
- net Net-(U1-GPIO1/RX): track 112.4 -> 63.5 mm
- net Net-(U1-GPIO2/SCK): track 92.5 -> 47.0 mm
- net Net-(U1-GPIO0/TX): track 99.7 -> 60.8 mm
- net Net-(U1-GPIO26/ADC0/A0): track 62.0 -> 23.6 mm
- net Net-(U1-GPIO4/MISO): track 110.0 -> 72.1 mm
- net +5V: track 138.3 -> 109.4 mm, vias 0 -> 3
- net Net-(D3-DIN): track 16.6 -> 35.8 mm
- net Net-(D4-K): track 30.6 -> 45.1 mm
- net Net-(D2-DIN): track 7.26 -> 5.75 mm
- net Net-(Q1-G): track 8.55 -> 7.73 mm
Other:
- board size 166.7 x 154.5 mm -> 107.9 x 100 mm

Commit message: uohewf
Parts:
- U1: footprint RF_Module:MCU_Seeed_ESP32C3 -> Seeed Studio XIAO Series Library:XIAO-RP2040-DIP
- moved U1 1.70 mm to (157.2, 133.3)
Routing:
- net Net-(U1-GPIO7/SCL): track 72.9 -> 47.2 mm
- net GND: track 252.7 -> 232.3 mm, vias 1 -> 0
- net Net-(D3-DIN): track 35.8 -> 15.9 mm
- net Net-(D4-K): track 45.1 -> 35.8 mm
- net +5V: track 109.4 -> 103.8 mm, vias 3 -> 0
- net Net-(U1-GPIO26/ADC0/A0): track 23.6 -> 18.7 mm
- net Net-(U1-GPIO28/ADC2/A2): track 47.6 -> 50.1 mm
- net Net-(Q1-G): track 7.73 -> 5.89 mm
- net Net-(U1-GPIO1/RX): track 63.5 -> 62.2 mm
- net Net-(U1-GPIO0/TX): track 60.8 -> 59.8 mm
- net Net-(D2-DIN): track 5.75 -> 4.75 mm
- net Net-(U1-GPIO4/MISO): track 72.1 -> 71.2 mm

Commit message: i hate this
Parts:
- removed D4: 1N4148, Diode_THT:D_DO-35_SOD27_P7.62mm_Horizontal
- added D1: SS14, Diode_SMD:D_SMA, F.Cu at (183.7, 126.2)
- added R2: 1kΩ, Resistor_SMD:R_0603_1608Metric, F.Cu at (169.9, 128.6)
- added R3: 1kΩ, Resistor_SMD:R_0603_1608Metric, F.Cu at (138.1, 133.3)
- D2, D3: value SK6812MINI -> LED; footprint LED_SMD:LED_SK6812MINI_PLCC4_3.5x3.5mm_P1.75mm -> LED_SMD:LED_0603_1608Metric
- moved D3 31.3 mm to (169.1, 133.3)
- moved C1 5.71 mm to (196.9, 114.3)
- moved D2 5.02 mm to (139.7, 128.6)
- moved R1 3.74 mm to (173.4, 129.9)
- moved M1 3.37 mm to (190.5, 114.1)
- moved SW6 2.72 mm to (140.7, 97.6)
- moved SW2 2.72 mm to (121.6, 100.0)
- moved SW4 2.70 mm to (159.7, 94.9)
- moved Q1 1.73 mm to (178.6, 133.3)
- moved U1 0.57 mm to (156.7, 133.0)
- moved SW1 0.36 mm to (126.2, 73.8)
- moved SW3 0.16 mm to (145.3, 71.1)
Connections:
- C1 pad 2: +5V -> +3.3V
- D2 pad 1: unconnected-(D2-DOUT-Pad1) -> Net-(D2-K)
- D2 pad 2: GND -> Net-(D2-A)
- D3 pad 1: Net-(D2-DIN) -> Net-(D3-K)
- D3 pad 2: GND -> Net-(D3-A)
- M1 pad 1: +5V -> +3.3V
- U1 pad 11: Net-(D3-DIN) -> Net-(D2-K)
- U1 pad 12: unconnected-(U1-3V3-Pad12)_1 -> +3.3V
- U1 pad 2: unconnected-(U1-GPIO27/ADC1/A1-Pad2) -> Net-(D3-A)
Routing:
- net +3.3V: track 0.00 -> 113.7 mm
- net +5V: track 103.8 -> 0.00 mm
- net Net-(D3-DIN): track 15.9 -> 0.00 mm
- net GND: track 232.3 -> 219.1 mm
- net Net-(D2-K): track 0.00 -> 9.58 mm
- net Net-(D1-K): track 35.8 -> 28.2 mm
- net Net-(D3-A): track 0.00 -> 6.06 mm
- net Net-(D2-A): track 0.00 -> 5.44 mm
- net Net-(D3-K): track 0.00 -> 5.09 mm
- net Net-(U1-GPIO26/ADC0/A0): track 18.7 -> 13.8 mm
- net Net-(D2-DIN): track 4.75 -> 0.00 mm
- net Net-(U1-GPIO7/SCL): track 47.2 -> 42.7 mm
- net Net-(U1-GPIO28/ADC2/A2): track 50.1 -> 46.7 mm
- net Net-(U1-GPIO4/MISO): track 71.2 -> 68.4 mm
- net Net-(U1-GPIO2/SCK): track 46.9 -> 44.3 mm
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
Commit message: everything's smaller now
Parts:
- moved SW6 21.5 mm to (161.5, 92.6)
- moved SW4 14.8 mm to (145.1, 92.6)
- moved D3 10.1 mm to (176.2, 126.2), turned to 0 degrees
- moved R2 9.01 mm to (175.4, 121.4), turned to 0 degrees
- moved SW2 8.85 mm to (126.4, 92.6)
- moved R3 7.53 mm to (145.3, 131.0), turned to -90 degrees
- moved U1 7.40 mm to (159.5, 126.2)
- moved D2 6.77 mm to (146.0, 126.2)
- moved M1 6.63 mm to (188.1, 108.0)
- moved C1 4.76 mm to (196.9, 109.5)
- moved SW1 3.50 mm to (128.4, 71.1)
- moved R1 3.45 mm to (173.0, 133.3)
- moved SW5 2.95 mm to (166.5, 71.1)
- moved D1 2.41 mm to (183.4, 123.8), turned to 0 degrees
- moved Q1 2.38 mm to (178.6, 131.0)
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Connections:
- U1 pad 14: +5V -> unconnected-(U1-VBUS-Pad14)_1
Routing:
- net +3.3V: track 113.7 -> 96.0 mm
- net GND: track 219.1 -> 202.6 mm
- net Net-(U1-GPIO4/MISO): track 68.4 -> 80.8 mm
- net Net-(U1-GPIO7/SCL): track 42.7 -> 31.0 mm
- net Net-(U1-GPIO0/TX): track 59.3 -> 47.8 mm
- net Net-(U1-GPIO26/ADC0/A0): track 13.8 -> 5.21 mm
- net Net-(D3-A): track 6.06 -> 11.1 mm
- net Net-(D1-K): track 28.2 -> 32.9 mm
- net Net-(D2-K): track 9.58 -> 5.09 mm
- net Net-(U1-GPIO1/RX): track 61.2 -> 57.3 mm
- net Net-(D2-A): track 5.44 -> 3.94 mm
- net Net-(U1-GPIO28/ADC2/A2): track 46.7 -> 45.4 mm
- net Net-(Q1-G): track 4.49 -> 5.20 mm
Other:
- board size 107.9 x 100 mm -> 98.1 x 90.9 mm

Commit message: turns out im sped
Parts:
- removed R2, R3: 1kΩ, Resistor_SMD:R_0603_1608Metric
- D2, D3: value LED -> SK6812MINI; footprint LED_SMD:LED_0603_1608Metric -> LED_SMD:LED_SK6812MINI_PLCC4_3.5x3.5mm_P1.75mm
- moved D3 33.3 mm to (142.9, 125.3)
- moved D2 5.72 mm to (142.9, 131.0), turned to 0 degrees
- moved Q1 5.32 mm to (176.2, 126.2), turned to -90 degrees
- moved SW4 3.15 mm to (143.0, 90.2)
- moved M1 2.78 mm to (190.5, 109.4)
- moved SW6 2.45 mm to (162.1, 90.2)
- moved D1 2.38 mm to (183.4, 121.4)
- moved SW2 2.38 mm to (126.4, 90.2)
- moved R1 0.83 mm to (173.8, 133.3)
- moved C1 0.78 mm to (197.6, 109.5)
- moved SW1 0.32 mm to (128.7, 71.1)
- moved SW3 0.32 mm to (147.8, 71.1)
- moved SW5 0.32 mm to (166.8, 71.1)
Connections:
- D2 pad 1: Net-(D2-K) -> Net-(D2-DOUT)
- D2 pad 2: Net-(D2-A) -> GND
- D3 pad 1: Net-(D3-K) -> unconnected-(D3-DOUT-Pad1)
- D3 pad 2: Net-(D3-A) -> GND
- U1 pad 11: Net-(D2-K) -> unconnected-(U1-GPIO3/MOSI-Pad11)_1
- U1 pad 14: unconnected-(U1-VBUS-Pad14)_1 -> +5V
- U1 pad 2: Net-(D3-A) -> Net-(D2-DIN)
Routing:
- net GND: track 202.6 -> 226.6 mm
- net Net-(D2-DIN): track 0.00 -> 23.5 mm
- net Net-(U1-GPIO4/MISO): track 80.8 -> 61.2 mm
- net +5V: track 0.00 -> 18.4 mm
- net Net-(D3-A): track 11.1 -> 0.00 mm
- net +3.3V: track 96.0 -> 85.1 mm
- net Net-(D2-DOUT): track 0.00 -> 5.34 mm
- net Net-(D2-K): track 5.09 -> 0.00 mm
- net Net-(D3-K): track 5.09 -> 0.00 mm
- net Net-(D2-A): track 3.94 -> 0.00 mm
- net Net-(Q1-G): track 5.20 -> 9.12 mm
- net Net-(U1-GPIO28/ADC2/A2): track 45.4 -> 48.7 mm
- net Net-(D1-K): track 32.9 -> 30.5 mm
- net Net-(U1-GPIO7/SCL): track 31.0 -> 33.2 mm
- net Net-(U1-GPIO26/ADC0/A0): track 5.21 -> 6.04 mm
