File: PCB/me.kicad_pcb (KiCad board)
At the start: 2 copper layers, 92.2 x 85.4 mm, 14 parts, among them M1 Motor_DC, Q1 AO3400A, SW1 SW_Push, SW2 SW_Push, SW3 SW_Push, SW4 SW_Push, SW5 SW_Push, SW6 SW_Push, U1 XIAO-RP2040-DIP

Commit message: delete
Routing:
- net GND: track 190.0 -> 209.1 mm
Changed lines of the file:
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@@
+	)
+	(segment
+		(start 152.55875 59.21375)
+		(end 161.925 59.21375)
+		(width 0.2)
+		(layer "F.Cu")
+		(net 1)
 	)
 	(segment
 		(start 144.625 113.425)
 		(end 149.0955 117.8955)
+		(width 0.2)
+		(layer "F.Cu")
+		(net 1)
+	)
+	(segment
+		(start 162.08375 78.26375)
+		(end 161.925 78.105)
 		(width 0.2)
 		(layer "F.Cu")
@@
 	)
 	(segment
+		(start 161.925 78.105)
+		(end 161.925 59.21375)
+		(width 0.2)
+		(layer "F.Cu")
+		(net 1)
+	)
+	(segment
 		(start 152.55875 59.21375)
 		(end 152.55875 78.1525)
@@
 	)
 	(segment
-		(start 152.55875 59.21375)
+		(start 161.925 59.21375)
 		(end 171.60875 59.21375)
 		(width 0.2)
